File: pcb/relow-pcb.sch (KiCad schematic (older format))
At the start: 71 parts, among them IC1 AD8495, IC2 ATMEGA328P_TQFP, IC3 FT230X_SOP, J1 MICROUSB, J2 TOASTER, K1 S212S01, P1 AVR_ISP, Q1 MMBT4401, Q2 MMBT4401, Q3 MMBT4401, Q4 MMBT4401, Q5 MMBT4401

Commit message: working on the board
Parts:
- ROT1: value ROTARY-ENCODER -> SET TEMP
Connections:
- net GND: now also Q2.2 (E); no longer Q2.3 (C)
- net MISO: now also R27.1; no longer R28.1
- net MOSI: now also R33.1; no longer R27.1
- net SCK: now also R28.1; no longer R30.1
- net SEGB: now also IC2.8 (XTAL2(PB7)); no longer IC2.13 (PB1(PCINT1/OC1A))
- net SEGG: now also IC2.13 (PB1(PCINT1/OC1A)); no longer IC2.7 (XTAL1(PB6))
- net VCC: now also LED1.2 (A), LED2.2 (A); no longer R5.2, R6.2
- net at J2.1: now also K1.1 (OUT2); no longer K1.2 (OUT1)
- net at J2.2: now also K1.2 (OUT1); no longer K1.1 (OUT2)
- net at K1.4 (IN-), R18.2: now also Q2.3 (C); no longer Q2.2 (E)
- net at IC3.14 (CBUS1): now also R5.1; no longer LED1.1 (C)
- net at IC3.7 (CBUS2): now also R6.1; no longer LED2.1 (C)
- removed net SEGDP: IC2.8 (XTAL2(PB7)), R33.1
- new net: LED1.1 (C), R5.2
- new net: LED2.1 (C), R6.2
- new net SEGF: IC2.7 (XTAL1(PB6)), R30.1
Other:
- moved on the sheet: LED1, LED2, R5, R6

Commit message: components placed. starting traces
Parts:
- R18: value 1kΩ -> 330Ω
Changed lines of the file:
@@
 U 1 1 5275F634
 P 8100 5850
-F 0 "R18" H 7950 5950 60  0000 C CNN
-F 1 "1kΩ" H 8150 5950 60  0000 C CNN
+F 0 "R18" H 7900 5950 60  0000 C CNN
+F 1 "330Ω" H 8150 5950 60  0000 C CNN
 F 2 "~" H 8100 5850 60  0000 C CNN
 F 3 "~" H 8100 5850 60  0000 C CNN

Commit message: layout done. ready to order (after triple checking)
Parts:
- IC2: value ATMEGA328P_TQFP -> ATMEGA328P
- IC3: value FT230X_SOP -> FT230X
- J1: value MICROUSB -> USB
- R1, R10, R11, R12, R14, R9: value 10kΩ_opt -> opt10kΩ
Connections:
- net GND: now also R13.1, R15.1; no longer LED3.1 (C), LED4.1 (C)
- net LED_START: now also LED3.2 (A); no longer R13.2
- net LED_STOP: now also LED4.2 (A); no longer R15.2
- new net: LED3.1 (C), R13.2
- new net: LED4.1 (C), R15.2
Other:
- moved on the sheet: LED3, LED4, R13, R15
Changed lines of the file:
@@
 L LED LED3
 U 1 1 5275FE41
-P 5850 4900
-F 0 "LED3" H 6000 5000 50  0000 C CNN
-F 1 "ON" H 5750 5000 50  0000 C CNN
-F 2 "~" H 5850 4900 60  0000 C CNN
-F 3 "~" H 5850 4900 60  0000 C CNN
-	1    5850 4900
+P 6250 4900
+F 0 "LED3" H 6350 5000 50  0000 C CNN
+F 1 "ON" H 6150 5000 50  0000 C CNN
+F 2 "~" H 6250 4900 60  0000 C CNN
+F 3 "~" H 6250 4900 60  0000 C CNN
+	1    6250 4900
 	-1   0    0    1
 $EndComp
@@
 L LED LED4
 U 1 1 5275FE91
-P 5850 5600
-F 0 "LED4" H 6000 5700 50  0000 C CNN
-F 1 "OFF" H 5750 5700 50  0000 C CNN
-F 2 "~" H 5850 5600 60  0000 C CNN
-F 3 "~" H 5850 5600 60  0000 C CNN
-	1    5850 5600
+P 6250 5600
+F 0 "LED4" H 6350 5700 50  0000 C CNN
+F 1 "OFF" H 6150 5700 50  0000 C CNN
+F 2 "~" H 6250 5600 60  0000 C CNN
+F 3 "~" H 6250 5600 60  0000 C CNN
+	1    6250 5600
 	-1   0    0    1
 $EndComp
@@
 L R R15
 U 1 1 52760134
-P 6250 5600
-F 0 "R15" H 6150 5500 60  0000 C CNN
-F 1 "180Ω" H 6400 5500 60  0000 C CNN
-F 2 "~" H 6250 5600 60  0000 C CNN
-F 3 "~" H 6250 5600 60  0000 C CNN
-	1    6250 5600
+P 5850 5600
+F 0 "R15" H 5600 5500 60  0000 C CNN
+F 1 "180Ω" H 5850 5500 60  0000 C CNN
+F 2 "~" H 5850 5600 60  0000 C CNN
+F 3 "~" H 5850 5600 60  0000 C CNN
+	1    5850 5600
 	1    0    0    -1
 $EndComp
@@
 L R R13
 U 1 1 5276015C
-P 6250 4900
-F 0 "R13" H 6150 4800 60  0000 C CNN
-F 1 "180Ω" H 6400 4800 60  0000 C CNN
-F 2 "~" H 6250 4900 60  0000 C CNN
-F 3 "~" H 6250 4900 60  0000 C CNN
-	1    6250 4900
+P 5850 4900
+F 0 "R13" H 5650 4800 60  0000 C CNN
+F 1 "180Ω" H 5900 4800 60  0000 C CNN
+F 2 "~" H 5850 4900 60  0000 C CNN
+F 3 "~" H 5850 4900 60  0000 C CNN
+	1    5850 4900
 	1    0    0    -1
 $EndComp
@@
 P 8250 2100
 F 0 "IC2" H 7550 3250 60  0000 C CNN
-F 1 "ATMEGA328P_TQFP" H 8600 900 60  0000 C CNN
+F 1 "ATMEGA328P" H 8600 900 60  0000 C CNN
 F 2 "~" H 8250 2100 60  0000 C CNN
 F 3 "~" H 8250 2100 60  0000 C CNN
@@
 P 7900 4250
 F 0 "R9" H 8000 4350 60  0000 C CNN
-F 1 "10kΩ_opt" H 7850 4450 60  0000 C CNN
+F 1 "opt10kΩ" H 7850 4450 60  0000 C CNN
 F 2 "~" H 7900 4250 60  0000 C CNN
 F 3 "~" H 7900 4250 60  0000 C CNN
@@
 P 6600 4700
 F 0 "R12" H 6350 4900 60  0000 C CNN
-F 1 "10kΩ_opt" H 6500 4800 60  0000 C CNN
+F 1 "opt10kΩ" H 6500 4800 60  0000 C CNN
 F 2 "~" H 6600 4700 60  0000 C CNN
 F 3 "~" H 6600 4700 60  0000 C CNN
@@
 P 6600 5400
 F 0 "R14" H 6400 5600 60  0000 C CNN
-F 1 "10kΩ_opt" H 6500 5500 60  0000 C CNN
+F 1 "opt10kΩ" H 6500 5500 60  0000 C CNN
 F 2 "~" H 6600 5400 60  0000 C CNN
 F 3 "~" H 6600 5400 60  0000 C CNN
@@
 P 9700 4250
 F 0 "R10" H 9450 4050 60  0000 C CNN
-F 1 "10kΩ_opt" H 9800 4050 60  0000 C CNN
+F 1 "opt10kΩ" H 9800 4050 60  0000 C CNN
 F 2 "~" H 9700 4250 60  0000 C CNN
 F 3 "~" H 9700 4250 60  0000 C CNN
@@
 P 9700 4350
 F 0 "R11" H 9450 4150 60  0000 C CNN
-F 1 "10kΩ_opt" H 9800 4150 60  0000 C CNN
+F 1 "opt10kΩ" H 9800 4150 60  0000 C CNN
 F 2 "~" H 9700 4350 60  0000 C CNN
 F 3 "~" H 9700 4350 60  0000 C CNN
@@
 P 1250 3900
 F 0 "J1" H 1100 3550 60  0000 C CNN
-F 1 "MICROUSB" H 1250 3450 60  0000 C CNN
+F 1 "USB" H 1250 3450 60  0000 C CNN
 F 2 "~" H 1150 3900 60  0000 C CNN
 F 3 "~" H 1150 3900 60  0000 C CNN
@@
 P 2950 3650
 F 0 "IC3" H 2700 4450 60  0000 C CNN
-F 1 "FT230X_SOP" H 3000 3100 60  0000 C CNN
+F 1 "FT230X" H 3000 3100 60  0000 C CNN
 F 2 "~" H 2950 3650 60  0000 C CNN
 F 3 "~" H 2950 3650 60  0000 C CNN
@@
 P 6600 1100
 F 0 "R1" H 6400 1000 60  0000 C CNN
-F 1 "10kΩ_opt" H 6750 1000 60  0000 C CNN
+F 1 "opt10kΩ" H 6750 1000 60  0000 C CNN
 F 2 "~" H 6600 1100 60  0000 C CNN
 F 3 "~" H 6600 1100 60  0000 C CNN

Commit message: going to bed again
Parts:
- C1, C10, C11, C12, C13, C2, C3, C4, C5, C6, C7, C8, C9, R1, R10, R11, R12, R13, R14, R15, R16, R17, R18, R19, R2, R20, R21, R22, R23, R24, R25, R26, R27, R28, R29, R3, R30, R31, R32, R33, R34, R35, R4, R5, R6, R7, R8, R9: footprint ~ -> 0603(1608m)
- F1: footprint ~ -> 1206(3216m); Manufacturer (none) -> Bel Fuse; Part (none) -> 0ZCJ0050FF2G
- IC1: footprint (none) -> MSOP8
- IC2: footprint ~ -> TQFP32_7mm; Manufacturer (none) -> AVR; Part (none) -> ATMEGA328P-AU
- IC3: footprint ~ -> SSOP16; Manufacturer (none) -> FTDI; Part (none) -> FT230XS-R
- J1: footprint ~ -> MICROUSB_sm; Manufacturer (none) -> FCI; Part (none) -> 10118192-0001LF
- J2: footprint ~ -> 2-PIN_SCREW-TERM_P200MIL; Manufacturer (none) -> On Shore Technology; Part (none) -> OSTTC022162
- K1: footprint ~ -> SHARP_SIP_SSR
- LED1, LED2: footprint ~ -> 0603(1608m)_led
- LED3, LED4, LED5: footprint ~ -> LED-5mm
- LED6: footprint (none) -> SF_4-DIGIT_7-SEGMENT_CC; Manufacturer (none) -> Sparkfun; Part (none) -> COM-11405
- P1: footprint ~ -> 2x3-array
- Q1, Q2, Q3, Q4, Q5: footprint ~ -> SOT23; Manufacturer (none) -> ON Semiconductor; Part (none) -> MMBT4401LT1G
- ROT1: footprint (none) -> SF_ROTARY-ENCODER; Manufacturer (none) -> Alpha; Part (none) -> RE130F-41-175F-12P
- S1, S2: footprint ~ -> SPST_4-pin-thru
- TC1: footprint (none) -> THERMOCOUPLE_MINI_PCC-SMP; Manufacturer (none) -> Newport Electronics; Part (none) -> PCC-SMP-K

Commit message: USB caps should be 47pF, not 47nF
Parts:
- C12, C13: value 47nF -> 47pF
Changed lines of the file:
@@
 P 1700 4100
 F 0 "C12" V 1500 4150 60  0000 C CNN
-F 1 "47nF" V 1400 4100 60  0000 C CNN
+F 1 "47pF" V 1400 4100 60  0000 C CNN
 F 2 "0603(1608m)" H 1700 4100 60  0001 C CNN
 F 3 "~" H 1700 4100 60  0000 C CNN
@@
 P 1900 4100
 F 0 "C13" V 1700 4050 60  0000 C CNN
-F 1 "47nF" V 1600 4000 60  0000 C CNN
+F 1 "47pF" V 1600 4000 60  0000 C CNN
 F 2 "0603(1608m)" H 1900 4100 60  0001 C CNN
 F 3 "~" H 1900 4100 60  0000 C CNN
