File: pcb/reflow-pcb.sch (KiCad schematic (older format))
At the start: 71 parts, among them IC1 AD8495, IC2 ATMEGA328P, IC3 FT230X, J1 USB, J2 TOASTER, K1 S212S01, P1 AVR_ISP, Q1 MMBT4401, Q2 MMBT4401, Q3 MMBT4401, Q4 MMBT4401, Q5 MMBT4401

Commit message: adding FTDI RTS cap. fixes #2
Parts:
- added C?: 0.1uF, ~, symbol C
Connections:
- wire segments 221 -> 224
Changed lines of the file:
@@
 Sheet 1 1
 Title "reflow pcb"
-Date "5 nov 2013"
+Date "20 jan 2014"
 Rev "0.1"
 Comp "Wiley Cousins, LLC."
@@
 Text Label 4000 3200 2    60   ~ 0
 USART_TX
-Text Label 4000 3300 2    60   ~ 0
+Text Label 3950 2900 0    60   ~ 0
 RESET
 $Comp
@@
 	4000 3200 3450 3200
 Wire Wire Line
-	3450 3300 4000 3300
-Wire Wire Line
 	3450 3700 3550 3700
 Wire Wire Line
@@
 Wire Wire Line
 	8450 6000 8550 6000
+$Comp
+L C C?
+U 1 1 52DD91E9
+P 4200 3100
+F 0 "C?" V 4100 2950 60  0000 C CNN
+F 1 "0.1uF" V 4000 2900 60  0000 C CNN
+F 2 "~" H 4200 3100 60  0001 C CNN
+F 3 "~" H 4200 3100 60  0001 C CNN
+	1    4200 3100
+	0    -1   -1   0
+$EndComp
+Wire Wire Line
+	3450 3300 4200 3300
+Wire Wire Line
+	4200 3300 4200 3200
+Wire Wire Line
+	4200 3000 4200 2900
+Wire Wire Line
+	4200 2900 3950 2900
 $EndSCHEMATC

Commit message: schematic first pass done. got that AC converter on board
Parts:
- removed C8: 0.1uF, 0603(1608m), symbol C
- removed Q1, Q3, Q4, Q5: MMBT4401, SOT23, symbol NPN-BJT_SOT
- removed R13, R15: 180Ω, 0603(1608m), symbol R
- removed R17, R22, R29, R34: 10kΩ, 0603(1608m), symbol R
- removed R19, R25, R31, R35: 1kΩ, 0603(1608m), symbol R
- added C? (x2): 22pF, ~, symbol C
- added C? (x4): 0.1uF, ~, symbol C
- added C?: 22uF, ~, symbol C_POL
- added C?: 100uF, ~, symbol C_POL
- added C?: 10uF, ~, symbol C
- added D? (x3): D, ~, symbol D
- added F?: 1.0A, ~, symbol FUSE
- added IC?: ULN2803A, ~, symbol ULN2803A
- added IC?: 74HC238, ~, symbol 74HC238
- added IC?: 74HC595, symbol 74HC595
- added IC?: LM1117, ~, symbol LM1117
- added J?: AC IN, ~, symbol 2PIN_FEMALE
- added L?: 1.0mH, ~, symbol L
- added LED?: CURRENT TEMP, SF_4-DIGIT_7-SEGMENT_CC, symbol 7-SEG_4-NUM-DISPLAY
- added PS?: BP5039B12, ~, symbol BP5039B12
- added R? (x3): 10kΩ, ~, symbol R
- added R? (x2): 330Ω, ~, symbol R
- added R?: 10Ω, ~, symbol R
- added RV?: VDR, ~, symbol VDR
- added Y?: 8MHz, ~, symbol CRYSTAL
- J2: value TOASTER -> HEATER
- LED6: value 7-SEG_4-NUM-DISPLAY -> TARGET TEMP
- R1, R10, R11, R12, R14, R9: value opt10kΩ -> 10kΩ
- R21, R24, R26, R27, R28, R30, R32, R33: value 180Ω -> 330Ω
Connections:
- net labels added: +12V, AC1, AC2, DIGA, DIGB, DIGC, DIGEN, HT, LAT, STAT_OFF, STAT_ON, VBUS
- net labels removed: DIG1, DIG2, DIG3, DIG4, LED_START, LED_STOP
- wire segments 224 -> 287
- no-connect marks 3 -> 6
Other:
- note added: "AC IN & 3.3V REGULATOR"
- note added: "DISPLAYS"
- note added: "SCREW TERMINALS"
- note added: "SWITCHES & STATUS"
- note removed: "DISPLAY"
- note removed: "SWITCH INPUTS"
- moved on the sheet: C1, C10, C11, C12, C13, C2, C3, C4, C5, C6, C7, C9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

Commit message: calling it a night
Parts:
- C18: renamed from C?; Manufacturer (none) -> Panasonic; Part (none) -> EEE-FT1E101AP
- C20: renamed from C?; Manufacturer (none) -> Samsung; Part (none) -> CL31B104KEHSFNE
- C21: renamed from C?; Manufacturer (none) -> Panasonic; Part (none) -> ECA-2EM220
- D1: renamed from D?; value D -> 1N5819
- D2: renamed from D?; value D -> 1N4001
- D3: renamed from D?; value D -> 1N4005
- L1: renamed from L?; Manufacturer (none) -> Bourns; Part (none) -> SRR1260-102K
- R16: value 180Ω -> 100Ω
- RV1: renamed from RV?; value VDR -> 185V; Manufacturer (none) -> Bourns; Part (none) -> MOV-07D201K
- gave numbers to parts that had none: 22
Connections:
- wire segments 287 -> 289

Commit message: schematic cleanup and component selection
Parts:
- removed C22: 10uF, ~, symbol C
- removed D1: 1N5819, ~, symbol D
- removed D2: 1N4001, ~, symbol D
- removed IC1: AD8495, MSOP8, symbol AD849X
- removed Q2: MMBT4401, SOT23, symbol NPN-BJT_SOT
- removed R1, R14, R23: 10kΩ, 0603(1608m), symbol R
- removed R20: 2.2kΩ, 0603(1608m), symbol R
- removed S2: STOP, SPST_4-pin-thru, symbol SPST
- added C22: 10uF, symbol C_POL
- added D2: PMEG4005CT, symbol SCHOTTKY_DUAL-CC
- added IC4: MAX31855, symbol MAX31855
- added Q1: DDTD113ZC, symbol NPN-BJT-BIASED_SOT
- added R27, R28: 10kΩ, symbol R
- added R6: 1MΩ, symbol R
- C11: renamed from C4; value 10uF -> 1uF
- C2: renamed from C11; value 10uF -> 0.1uF
- C7: renamed from C2; value 1uF -> 0.1uF
- C8: renamed from C5; value 1uF -> 0.1uF
- IC7: Link (none) -> http://www.digikey.com/product-detail/en/AZ1117CH-3.3TRG1/A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; Manufacturer (none) -> Diodes Incorporated; Part (none) -> AZ1117CH-3.3TRG1
- LED3: renamed from LED6; Link (none) -> http://www.digikey.com/product-detail/en/LTC-5723HR/160-187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; Manufacturer Sparkfun -> Lite-On; Part COM-11405 -> LTC-5723HR
- LED4: renamed from LED7; Link (none) -> http://www.digikey.com/product-detail/en/LTC-5723HR/160-187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; Manufacturer Sparkfun -> Lite-On; Part COM-11405 -> LTC-5723HR
- PS1: Link (none) -> http://www.digikey.com/product-search/en?mpart=BP5039B12; Manufacturer (none) -> Bourns; Part (none) -> BP5039B12
- R10: renamed from R2; value 4.7kΩ -> 330Ω
- R11: renamed from R3; value 4.7kΩ -> 330Ω
- S1: value START -> START/STOP
- renumbered C12 to C1, C1 to C10, C15 to C12, C3 to C13, C6 to C14, C7 to C15, C13 to C3, C9 to C4, C10 to C5, C8 to C6, C14 to C9, D3 to D1, IC3 to IC1, IC4 to IC2, IC5 to IC3, IC6 to IC5, IC2 to IC6, J3 to J2, J2 to J3, LED4 to LED1, LED3 to LED2, LED1 to LED5, LED2 to LED6, LED5 to LED7, R13 to R1, R17 to R12, R19 to R13, R22 to R14, R16 to R15, R18 to R16, R21 to R19, R15 to R2, R24 to R20, R26 to R21, R27 to R22, R28 to R23, R30 to R24, R32 to R25, R33 to R26, R12 to R3, R9 to R30, R25 to R31, R11 to R32, R10 to R33, R7 to R4, R8 to R5, R4 to R7, R5 to R8, R6 to R9
Connections:
- net labels added: DISP_CS, ST_SP, TEMP_CS
- net labels removed: LAT, START, STOP, TEMP
- wire segments 289 -> 276
- no-connect marks 6 -> 7
Other:
- moved on the sheet: C10, C11, C19, C7, C8, R10, R11, R3, R7, S1, TC1

Commit message: some schematic work.
Parts:
- removed C22: 10uF, symbol C_POL
- removed C7, C8: 0.1uF, 0603(1608m), symbol C
- removed R10, R11: 330Ω, 0603(1608m), symbol R
- removed R6: 1MΩ, symbol R
- removed R7: 1MΩ, 0603(1608m), symbol R
- added C?: 22uF, symbol C
- added C?: 0.1uF, symbol C
- added FB? (x2): FB, symbol FB
- C11: value 1uF -> 10nF
- C19: value 0.1uF -> 10uF
Connections:
- net GND: now also C?.1, C?.1
- net VCC: now also C?.2; no longer IC6.20 (AREF)
- net at TC1.1 (T+): now also FB?.1
- net at TC1.2 (T-): now also FB?.1
- net at C11.1, IC4.2 (T-): now also FB?.2
- net at C11.2, IC4.3 (T+): now also FB?.2
- new net: C?.2, IC6.20 (AREF)
Other:
- moved on the sheet: C10, C11, C13, C14, C15, IC4, TC1

Commit message: preparing for new layout
Parts:
- removed C2: 0.1uF, 0603(1608m), symbol C
- removed IC2: ULN2803A, ~, symbol ULN2803A
- removed IC3: 74HC238, ~, symbol 74HC238
- removed LED3: TARGET TEMP, SF_4-DIGIT_7-SEGMENT_CC, symbol 7-SEG_4-NUM-DISPLAY
- removed LED4: CURRENT TEMP, SF_4-DIGIT_7-SEGMENT_CC, symbol 7-SEG_4-NUM-DISPLAY
- removed Q1: DDTD113ZC, symbol NPN-BJT-BIASED_SOT
- removed R12: 10kΩ, ~, symbol R
- removed R2: 330Ω, ~, symbol R
- removed R3: 10kΩ, 0603(1608m), symbol R
- removed S1: START/STOP, SPST_4-pin-thru, symbol SPST
- added C12: 10uF, symbol C
- added IC2: CD4028, symbol CD4028
- added LED3, LED4: 7-SEGMENT, symbol 7-SEG-4-DIG-DP+CLK_CC-LED
- added Q1, Q10, Q11, Q2, Q3, Q4, Q5, Q6, Q7, Q8, Q9: 2N7002, symbol N-CHAN-MOSFET_SOT
- added R17, R18, R4: 10kΩ, 0603(1608m), symbol R
- added R23: 10kΩ, symbol R
- added ROT2: KNOB, SF_ROTARY-ENCODER, symbol ROTARY-ENCODER
- C10: renamed from C16; value 22pF -> 24pF
- C11: renamed from C17; value 22pF -> 24pF
- C3: renamed from C18; Distrib. Link (none) -> http://www.digikey.com/product-detail/en/EEE-FT1E101AP/PCE5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; Distrib. Part (none) -> PCE5007CT-ND; Distributor (none) -> Digikey; Manuf. Part (none) -> EEE-FT1E101AP; Part EEE-FT1E101AP -> (none)
- C5: renamed from C20; Distrib. Link (none) -> http://www.digikey.com/product-detail/en/CL31B104KEHSFNE/12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; Distrib. Part (none) -> 1276-3083-1-ND; Distributor (none) -> Digikey; Manuf. Part (none) -> CL31B104KEHSFNE; Part CL31B104KEHSFNE -> (none)
- C6: renamed from C21; Distrib. Link (none) -> http://www.digikey.com/product-detail/en/EEU-EE2E220/P13640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; Distrib. Part (none) -> P13640-ND; Distributor (none) -> Digikey; Manuf. Part (none) -> EEU-EE2E220; Manufacturer Panasonic -> Panasonic Electronic Components; Part ECA-2EM220 -> (none)
- D2: renamed from D1; value 1N4005 -> S1J-13-F; Distrib. Link (none) -> http://www.digikey.com/product-detail/en/S1J-13-F/S1J-FDICT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; Distrib. Part (none) -> S1J-FDICT-ND; Distributor (none) -> Digikey; Manuf. Part (none) -> S1J-13-F; Manufacturer (none) -> Diodes Incorporated
- L1: Distrib. Link (none) -> http://www.digikey.com/product-detail/en/SRR1260-102K/SRR12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; Distrib. Part (none) -> SRR1260-102KCT-ND; Distributor (none) -> Digikey; Manuf. Part (none) -> SRR1260-102K; Part SRR1260-102K -> (none)
- LED1: value OFF -> RED
- LED2: value ON -> GRN
- LED5: renamed from LED7; value HOT -> RED
- R21: renamed from R31; Distrib. Link (none) -> http://www.digikey.com/product-detail/en/RC1206FR-0710RL/31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; Distrib. Part (none) -> 311-10.0FRCT-ND; Distributor (none) -> Digikey; Manuf. Part (none) -> RC1206FR-0710RL; Manufacturer (none) -> Yageo
- ROT1: value SET TEMP -> KNOB
- VR1: renamed from RV1; value 185V -> 240V; Distrib. Part (none) -> MOV-14D241K-ND; Distributor (none) -> Digikey; Manuf. Part (none) -> MOV-14D241K; Part MOV-07D201K -> (none)
- gave numbers to parts that had none: 4
- renumbered C12 to C1, C1 to C17, C3 to C18, C4 to C19, C9 to C2, C5 to C20, C6 to C21, C19 to C4, C10 to C8, C11 to C9, D2 to D1, F2 to F1, F1 to F2, IC5 to IC1, IC7 to IC3, IC6 to IC5, IC1 to IC6, J2 to J1, J3 to J2, J1 to J3, LED5 to LED6, LED6 to LED7, R27 to R1, R22 to R10, R23 to R11, R24 to R12, R25 to R13, R26 to R14, R33 to R15, R32 to R16, R15 to R19, R13 to R2, R16 to R20, R28 to R22, R4 to R24, R5 to R25, R8 to R26, R9 to R27, R30 to R3, R14 to R5, R1 to R6, R19 to R7, R20 to R8, R21 to R9
Connections:
- net STAT_ON is gone; now on net STAT_2: IC5.11 (PD7(PCINT23/AIN1))
- net DIGA: now also IC2.10 (A)
- net DIGB: now also IC2.13 (B)
- net DIGC: now also IC2.12 (C)
- net ENC_A: now also R15.1; no longer R15.2
- net ENC_B: now also R16.1; no longer R16.2
- net GND: now also C12.1, IC2.8 (VSS), Q1.2 (S), Q10.2 (S), Q11.2 (S), Q2.2 (S), Q3.2 (S), Q4.2 (S), Q5.2 (S), Q6.2 (S), Q7.2 (S), Q8.2 (S), Q9.2 (S), ROT2.3 (C), ROT2.5 (SW2); no longer LED1.1 (C), LED2.1 (C)
- net HEAT: now also Q11.1 (G)
- net RESET: now also R23.2
- net SEGA: now also R14.1, LED3.14 (A(L1)), LED4.14 (A(L1)); no longer R7.1
- net SEGB: now also R13.1, LED3.16 (B(L2)), LED4.16 (B(L2)); no longer R8.1
- net SEGC: now also R12.1, LED3.13 (C(L3)), LED4.13 (C(L3)); no longer R9.1
- net SEGD: now also R11.1, LED3.3 (D), LED4.3 (D); no longer R10.1
- net SEGDP: now also R7.1, LED3.7 (DP), LED4.7 (DP); no longer R14.1
- net SEGE: now also R10.1, LED3.5 (E), LED4.5 (E); no longer R11.1
- net SEGF: now also R9.1, LED3.11 (F), LED4.11 (F); no longer R12.1
- net SEGG: now also R8.1, LED3.15 (G), LED4.15 (G); no longer R13.1
- net TEMP_CS: now also IC5.2 (PD4(PCINT20/XCK/T0)); no longer IC5.13 (PB1(PCINT1/OC1A))
- net VBUS: now also F2.1; no longer F2.2
- net VCC: now also R15.2, R16.2, IC2.16 (VDD), R17.2, R18.2, R23.1, R4.2; no longer R15.1, R16.1
- net at K1.4 (IN-), R20.2: now also Q11.3 (D)
- net STAT_1: now reaches LED2.2 (A)
- net STAT_1: now also IC5.10 (PD6(PCINT22/OC0A/AIN0)), LED1.1 (C)
- net at LED1.2 (A), R6.1: now also LED2.1 (C)
- net at R7.2: now also IC1.7 (QH); no longer IC1.9 (QH')
- net at R8.2: now also IC1.6 (QG)
- net at R9.2: now also IC1.5 (QF); no longer IC1.7 (QH)
- net at R10.2: now also IC1.4 (QE); no longer IC1.6 (QG)
- net at R11.2: now also IC1.3 (QD); no longer IC1.5 (QF)
- net at R12.2: now also IC1.2 (QC); no longer IC1.4 (QE)
- net at R13.2: now also IC1.1 (QB); no longer IC1.3 (QD)
- net at R14.2: now also IC1.15 (QA); no longer IC1.2 (QC)
- net ENC_C: now reaches IC5.12 (PB0(PCINT0/CLKO/ICP1))
- net ENC_C: now also R17.1, ROT2.2 (A)
- net at J3.1 (VBUS): now also F2.2, C12.2; no longer F2.1
- net DIGEN renamed DIGD
- net DIGD: now also IC2.11 (D)
- net SET renamed SW_TEMP
- net STAT_OFF renamed STAT_2
- net STAT_2: no longer IC5.10 (PD6(PCINT22/OC0A/AIN0))
- net ST_SP renamed SW_TIME
- net SW_TIME: now also R4.1, ROT2.1 (SW1)
- new net: LED3.1 (DIG1), Q5.3 (D)
- new net: LED3.2 (DIG2), Q4.3 (D)
- new net: LED3.4 (L), Q3.3 (D)
- new net: LED3.6 (DIG3), Q2.3 (D)
- new net: LED3.8 (DIG4), Q1.3 (D)
- new net: LED4.8 (DIG4), Q6.3 (D)
- new net: LED4.6 (DIG3), Q7.3 (D)
- new net: LED4.4 (L), Q8.3 (D)
- new net: LED4.2 (DIG2), Q9.3 (D)
- new net: LED4.1 (DIG1), Q10.3 (D)
- new net DIG0: IC2.3 (Y0), Q10.1 (G)
- new net DIG1: IC2.14 (Y1), Q9.1 (G)
- new net DIG2: IC2.15 (Y3), Q7.1 (G)
- new net DIG3: IC2.1 (Y4), Q6.1 (G)
- new net DIG4: IC2.6 (Y5), Q5.1 (G)
- new net DIG5: IC2.7 (Y6), Q4.1 (G)
- new net DIG6: IC2.9 (Y8), Q2.1 (G)
- new net DIG7: IC2.5 (Y9), Q1.1 (G)
- new net ENC_D: IC5.13 (PB1(PCINT1/OC1A)), R18.1, ROT2.4 (B)
- new net L0: IC2.2 (Y2), Q8.1 (G)
- new net L1: IC2.4 (Y7), Q3.1 (G)
- no-connect marks 7 -> 5
Other:
- note added: "AC in and 3.3V regulator"
- note added: "AC relay"
- note added: "AC terminals"
- note added: "ATMega328p microcontroller"
- note added: "USB programming and debugging"
- note added: "displays"
- note added: "status indicators"
- note added: "thermocouple jack and amplifier"
- note added: "user input"
- note removed: "AC IN & 3.3V REGULATOR"
- note removed: "AC RELAY"
- note removed: "DISPLAYS"
- note removed: "MCU"
- note removed: "PROGRAMMING AND DEBUGGING"
- note removed: "SCREW TERMINALS"
- note removed: "SET TEMPERATURE INPUT"
- note removed: "SWITCHES & STATUS"
- note removed: "THERMOCOUPLE INPUT"
- moved on the sheet: C1, C10, C11, C13, C14, C15, C16, C17, C18, C19, C2, C20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

Commit message: work on layout
Parts:
- removed PS1: BP5039B12, ~, symbol BP5039B12
- added PS1: BP5037B12, symbol BP5037B12
- added S1: RST, symbol SPST
- F1: Distrib. Link (none) -> http://www.digikey.com/product-detail/en/C1Q%201/507-1077-1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; Distrib. Part (none) -> 507-1077-1-ND; Distributor (none) -> Digikey; Manuf. Part (none) -> C1Q 1; Manufacturer (none) -> Bel Fuse Inc
Connections:
- net +12V: now also PS1.1 (12V)
- net AC1: now also J1.2; no longer J1.1
- net GND: now also J1.1, J2.2, PS1.7 (COMMON), S1.1; no longer J1.2, J2.1
- net HT: now also J2.1; no longer J2.2
- net RESET: now also S1.2
- net at F1.1: now also PS1.10 (AC_IN)
- net at L1.2: now also PS1.3 (CHOKE)
- net at L1.1: now also PS1.5 (CHOKE)
Other:
- moved on the sheet: R23
Changed lines of the file:
@@
 Text Notes 9050 5950 0    100  ~ 0
 AC terminals
+Text Label 10000 6300 2    60   ~ 0
+AC1
 Text Label 10000 6200 2    60   ~ 0
-AC1
-Text Label 10000 6400 2    60   ~ 0
 AC2
-Text Label 10000 6600 2    60   ~ 0
+Text Label 10000 6500 2    60   ~ 0
 HT
 Text Label 10000 4600 2    60   ~ 0
@@
 Text Label 10000 4800 2    60   ~ 0
 HT
-$Comp
-L BP5039B12 PS1
-U 1 1 52DEDB79
-P 7750 1950
-F 0 "PS1" H 7550 2350 60  0000 C CNN
-F 1 "BP5039B12" H 7750 1500 60  0000 C CNN
-F 2 "~" H 7750 1950 60  0000 C CNN
-F 3 "~" H 7750 1950 60  0000 C CNN
-F 4 "Bourns" H 7750 1950 60  0001 C CNN "Manufacturer"
-F 5 "BP5039B12" H 7750 1950 60  0001 C CNN "Part"
-F 6 "http://www.digikey.com/product-search/en?mpart=BP5039B12" H 7750 1950 60  0001 C CNN "Link"
-	1    7750 1950
-	1    0    0    -1
-$EndComp
 Text Label 10000 1700 2    60   ~ 0
 AC1
@@
 F 2 "~" H 8450 1700 60  0000 C CNN
 F 3 "~" H 8450 1700 60  0000 C CNN
+F 4 "Bel Fuse Inc" H 8450 1700 60  0001 C CNN "Manufacturer"
+F 5 "C1Q 1" H 8450 1700 60  0001 C CNN "Manuf. Part"
+F 6 "Digikey" H 8450 1700 60  0001 C CNN "Distributor"
+F 7 "507-1077-1-ND" H 8450 1700 60  0001 C CNN "Distrib. Part"
+F 8 "http://www.digikey.com/product-detail/en/C1Q%201/507-1077-1-ND/615050" H 8450 1700 60  0001 C CNN "Distrib. Link"
 	1    8450 1700
 	1    0    0    -1
@@
 L R R23
 U 1 1 5392B750
-P 11950 1650
-F 0 "R23" H 11950 1500 60  0000 C CNN
-F 1 "10kΩ" H 11950 1400 60  0000 C CNN
-F 2 "" H 11950 1650 60  0001 C CNN
-F 3 "" H 11950 1650 60  0001 C CNN
-	1    11950 1650
+P 11950 1800
+F 0 "R23" H 11950 1650 60  0000 C CNN
+F 1 "10kΩ" H 11950 1550 60  0000 C CNN
+F 2 "" H 11950 1800 60  0001 C CNN
+F 3 "" H 11950 1800 60  0001 C CNN
+	1    11950 1800
 	1    0    0    -1
 $EndComp
@@
 L VCC #PWR055
 U 1 1 5392BB29
-P 11700 1650
-F 0 "#PWR055" H 11700 1750 30  0001 C CNN
-F 1 "VCC" H 11700 1750 30  0000 C CNN
-F 2 "" H 11700 1650 60  0000 C CNN
-F 3 "" H 11700 1650 60  0000 C CNN
-	1    11700 1650
+P 11700 1800
+F 0 "#PWR055" H 11700 1900 30  0001 C CNN
+F 1 "VCC" H 11700 1900 30  0000 C CNN
+F 2 "" H 11700 1800 60  0000 C CNN
+F 3 "" H 11700 1800 60  0000 C CNN
+	1    11700 1800
 	0    -1   -1   0
 $EndComp
@@
 	10250 6750 9000 6750
 Wire Wire Line
-	10000 6600 9750 6600
-Connection ~ 9800 6400
-Wire Wire Line
-	9800 6500 9750 6500
-Wire Wire Line
-	9800 6300 9750 6300
-Wire Wire Line
-	9800 6300 9800 6500
-Wire Wire Line
-	10000 6400 9800 6400
+	10000 6500 9750 6500
 Wire Wire Line
 	10000 6200 9750 6200
+Wire Wire Line
+	10000 6300 9750 6300
 Wire Notes Line
 	1250 1250 4500 1250
@@
 Connection ~ 8850 4750
 Wire Wire Line
-	11700 1650 11800 1650
+	11700 1800 11800 1800
 Wire Wire Line
 	12500 2350 12400 2350
@@
 Connection ~ 13350 6150
 Wire Wire Line
-	13350 6550 13350 6350
+	13350 6350 13350 6550
 Connection ~ 13350 6450
 Connection ~ 12150 6450
@@
 Wire Wire Line
 	12650 6850 12650 6750
+$Comp
+L SPST S1
+U 1 1 538F998D
+P 11950 1650
+F 0 "S1" H 11950 1850 60  0000 C CNN
+F 1 "RST" H 11950 1750 60  0000 C CNN
+F 2 "" H 11950 1650 60  0001 C CNN
+F 3 "" H 11950 1650 60  0001 C CNN
+	1    11950 1650
+	1    0    0    -1
+$EndComp
+$Comp
+L GND #PWR061
+U 1 1 538F9C4D
+P 11700 1650
+F 0 "#PWR061" H 11700 1650 30  0001 C CNN
+F 1 "GND" H 11700 1580 30  0001 C CNN
+F 2 "" H 11700 1650 60  0000 C CNN
+F 3 "" H 11700 1650 60  0000 C CNN
+	1    11700 1650
+	0    1    1    0
+$EndComp
+Wire Wire Line
+	11800 1650 11700 1650
+Wire Wire Line
+	12100 1800 12200 1800
+Wire Wire Line
+	12200 1800 12200 1650
+Connection ~ 12200 1650
+Text Label 10000 6600 2    60   ~ 0
+AC2
+Wire Wire Line
+	10000 6600 9750 6600
+$Comp
+L BP5037B12 PS1
+U 1 1 538FE1CA
+P 7750 1950
+F 0 "PS1" H 7550 2350 60  0000 C CNN
+F 1 "BP5037B12" H 7750 1500 60  0000 C CNN
+F 2 "" H 7450 2250 60  0001 C CNN
+F 3 "" H 7550 2350 60  0001 C CNN
+F 4 "Rohm Semiconductor" H 7650 2450 60  0001 C CNN "Manufacturer"
+F 5 "BP5037B12" H 7750 2550 60  0001 C CNN "Manuf. Part"
+F 6 "Digikey" H 7750 1950 60  0001 C CNN "Distributor"
+F 7 "BP5037B12-ND" H 7750 1950 60  0001 C CNN "Distrib. Part"
+F 8 "http://www.digikey.com/product-detail/en/BP5037B12/BP5037B12-ND/658553" H 7750 1950 60  0001 C CNN "Distrib. Link"
+	1    7750 1950
+	1    0    0    -1
+$EndComp
 $EndSCHEMATC
