File: pcb/reflow-pcb.kicad_pcb (KiCad board)
At the start: 2 copper layers, 76.2 x 44.5 mm, 75 parts, among them IC1 AD8495, IC2 ATMEGA328P, IC3 FT230X, J1 USB, J2 TOASTER, K1 S212S01, M3 VAL**, P1 AVR_ISP, Q1 MMBT4401, Q2 MMBT4401, Q3 MMBT4401, Q4 MMBT4401, Q5 MMBT4401

Commit message: how about i spell "reflow" correctly?
Routing:
- net VCC: track 245.8 -> 272.0 mm, vias 3 -> 5
Changed lines of the file:
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@@
     (thickness 1.6)
     (drawings 37)
-    (tracks 1026)
+    (tracks 1036)
     (zones 0)
     (modules 75)
@@
   )
   (layers
-    (15 F.Cu signal)
-    (0 B.Cu signal hide)
+    (15 F.Cu signal hide)
+    (0 B.Cu signal)
     (16 B.Adhes user)
     (17 F.Adhes user)
     (18 B.Paste user)
     (19 F.Paste user)
-    (20 B.SilkS user hide)
-    (21 F.SilkS user)
+    (20 B.SilkS user)
+    (21 F.SilkS user hide)
     (22 B.Mask user)
     (23 F.Mask user)
@@
     (pad_to_mask_clearance 0.0762)
     (aux_axis_origin 116.205 122.555)
-    (visible_elements 7FFFBFFF)
+    (visible_elements 7FFFDFFF)
     (pcbplotparams
       (layerselection 284196865)
@@
   (segment (start 148.6916 85.9536) (end 149.4282 85.217) (width 0.254) (layer F.Cu) (net 63))
   (segment (start 148.6916 90.4494) (end 148.6916 85.9536) (width 0.254) (layer F.Cu) (net 63))
+  (segment (start 159.447 119.126) (end 159.447 121.477) (width 0.254) (layer F.Cu) (net 64))
+  (segment (start 181.3814 121.0056) (end 181.3814 119.6086) (width 0.254) (layer F.Cu) (net 64))
+  (segment (start 180.848 121.539) (end 181.3814 121.0056) (width 0.254) (layer F.Cu) (net 64))
+  (segment (start 175.768 121.539) (end 180.848 121.539) (width 0.254) (layer F.Cu) (net 64))
+  (segment (start 175.641 121.412) (end 175.768 121.539) (width 0.254) (layer F.Cu) (net 64))
+  (via (at 175.641 121.412) (size 0.762) (layers F.Cu B.Cu) (net 64))
+  (segment (start 159.512 121.412) (end 175.641 121.412) (width 0.254) (layer B.Cu) (net 64))
+  (segment (start 159.385 121.539) (end 159.512 121.412) (width 0.254) (layer B.Cu) (net 64))
+  (via (at 159.385 121.539) (size 0.762) (layers F.Cu B.Cu) (net 64))
+  (segment (start 159.447 121.477) (end 159.385 121.539) (width 0.254) (layer F.Cu) (net 64))
   (segment (start 154.16784 89.89822) (end 155.27782 89.89822) (width 0.254) (layer F.Cu) (net 64))
   (segment (start 155.4734 91.27236) (end 155.24988 91.49588) (width 0.254) (layer F.Cu) (net 64))
@@
   (segment (start 158.623 119.126) (end 157.9118 118.4148) (width 0.254) (layer F.Cu) (net 64))
   (segment (start 180.278 119.888) (end 181.102 119.888) (width 0.254) (layer F.Cu) (net 64))
+  (segment (start 181.102 119.888) (end 181.3814 119.6086) (width 0.254) (layer F.Cu) (net 64))
   (segment (start 181.0512 117.856) (end 180.278 117.856) (width 0.254) (layer F.Cu) (net 64))
   (segment (start 181.3814 118.1862) (end 181.3306 118.1354) (width 0.254) (layer F.Cu) (net 64))
-  (segment (start 181.3306 118.1354) (end 181.0512 117.856) (width 0.254) (layer F.Cu) (net 64))
   (segment (start 181.3814 119.6086) (end 181.3814 118.1862) (width 0.254) (layer F.Cu) (net 64))
-  (segment (start 181.102 119.888) (end 181.3814 119.6086) (width 0.254) (layer F.Cu) (net 64))
+  (segment (start 181.3306 118.1354) (end 181.0512 117.856) (width 0.254) (layer F.Cu) (net 64))
   (segment (start 154.16784 89.89822) (end 152.53462 89.89822) (width 0.254) (layer F.Cu) (net 64))
   (segment (start 152.2984 89.662) (end 151.576 89.662) (width 0.254) (layer F.Cu) (net 64))

Commit message: work on layout
Parts:
- removed M3 (x4): VAL**, M3
- removed R28, R30, R32, R33: 180Ω, 0603(1608m)
- removed R29, R34: 10kΩ, 0603(1608m)
- removed R31, R35: 1kΩ, 0603(1608m)
- removed S2: STOP, SPST_4-pin-thru
- added C14: 0.1uF, capacitor:0603(1608m)-CHIP-CAP, F.Cu at (231.7, 136.8)
- added C15: 0.1uF, capacitor:0603(1608m)-CHIP-CAP, F.Cu at (253.2, 114.8)
- added C16: 0.1uF, capacitor:0603(1608m)-CHIP-CAP, F.Cu at (258.6, 108.4)
- added C17: 47pF, capacitor:0603(1608m)-CHIP-CAP, F.Cu at (175.0, 37.5)
- added C18: 47pF, capacitor:0603(1608m)-CHIP-CAP, F.Cu at (170.4, 37.5)
- added C19: 0.1uF, capacitor:0603(1608m)-CHIP-CAP, F.Cu at (178.3, 43.4)
- added C20: 0.1uF, capacitor:0603(1608m)-CHIP-CAP, F.Cu at (178.3, 41.9)
- added C21: 0.1uF, capacitor:0603(1608m)-CHIP-CAP, F.Cu at (240.5, 125.7)
- added D1: PMEG4005CT, sot:SOT23, F.Cu at (124.5, 112.4)
- added D2: S1J-13-F, diode:DO-214AC, F.Cu at (154.3, 116.2)
- added F2: 500mA, resistor:1206(3216m)-CHIP-RESISTOR, F.Cu at (179.3, 37.7)
- added FB1: FB, resistor:0603(1608m)-CHIP-RESISTOR, F.Cu at (203.0, 126.1)
- added FB2: FB, resistor:0603(1608m)-CHIP-RESISTOR, F.Cu at (244.3, 128.4)
- added IC4: MAX31855, soic:SOIC8, F.Cu at (74.9, 54.6)
- added IC5: ATMEGA328P, qfp:TQFP32_P0.8mm, F.Cu at (158.1, 41.9)
- added IC6: FT230X, sop:SSOP16, F.Cu at (172.7, 41.9)
- added J3: USB, connect-sm:MICROUSB_sm, F.Cu at (172.7, 31.8)
- added L1: 1.0mH, inductor:SM-INDUCTOR_12.5mmX12.5mm, F.Cu at (148.0, 107.3)
- added LED7: RXLED, led:0603(1608m)-SM-LED, F.Cu at (170.2, 47.6)
- added PS1: BP5037B12, rohm:ROHM-BP5037B12_SIP10_AC-DC, F.Cu at (136.5, 115.6)
- added Q10: 2N7002, sot:SOT23, F.Cu at (116.2, 53.3)
- added Q11: 2N7002, sot:SOT23, F.Cu at (160.7, 104.8)
- added Q6: 2N7002, sot:SOT23, F.Cu at (131.4, 53.3)
- added Q7: 2N7002, sot:SOT23, F.Cu at (127.6, 53.3)
- added Q8: 2N7002, sot:SOT23, F.Cu at (123.8, 53.3)
- added Q9: 2N7002, sot:SOT23, F.Cu at (120.0, 53.3)
- added ROT2: KNOB, sparkfun:SF-ROTARY-ENCODER, F.Cu at (94.0, 51.4)
- added VR1: 240V, bourns:BOURNS-MOV-14DxxxK_THRU-VARISTOR, F.Cu at (154.9, 124.5)
- added Y1: 8MHz, crystal:ABRACON-ABM2_xtal, F.Cu at (158.1, 32.4)
- C1, C8: footprint 0603(1608m) -> capacitor:0603(1608m)-CHIP-CAP
- C10: value 0.1uF -> 24pF; footprint 0603(1608m) -> capacitor:0603(1608m)-CHIP-CAP
- C11: value 10uF -> 24pF; footprint 0603(1608m) -> capacitor:0603(1608m)-CHIP-CAP
- C12: value 47pF -> 10uF; footprint 0603(1608m) -> capacitor:0805(2012m)-CHIP-CAP
- C13: value 47pF -> 0.1uF; footprint 0603(1608m) -> capacitor:0603(1608m)-CHIP-CAP
- C2: value 1uF -> 0.1uF; footprint 0603(1608m) -> capacitor:0603(1608m)-CHIP-CAP
- C3: value 0.1uF -> 100uF; footprint 0603(1608m) -> capacitor:PANA-D_CHEMI-F_6.3mm-SM-ALUMINUM
- C4: footprint 0603(1608m) -> capacitor:0805(2012m)-CHIP-CAP
- C5: value 1uF -> 0.1uF; footprint 0603(1608m) -> capacitor:1206(3216m)-CHIP-CAP
- C6: value 0.1uF -> 22uF; footprint 0603(1608m) -> capacitor:10mm-THRU-ALUMINUM-CAP
- C7: value 0.1uF -> 22uF; footprint 0603(1608m) -> capacitor:0805(2012m)-CHIP-CAP
- C9: value 0.1uF -> 10nF; footprint 0603(1608m) -> capacitor:0603(1608m)-CHIP-CAP
- F1: value 500mA -> 1.0A; footprint 1206(3216m) -> resistor:1206(3216m)-CHIP-RESISTOR
- IC1: value AD8495 -> 74HC595; footprint MSOP8 -> sop:TSSOP16
- IC2: value ATMEGA328P -> CD4028; footprint TQFP32_7mm -> sop:TSSOP16
- IC3: value FT230X -> LM1117; footprint SSOP16 -> sot:SOT223
- J1: value USB -> AC IN; footprint MICROUSB_sm -> connect-thru:1x2-SCREW-TERM_P200mil
- J2: value TOASTER -> HEATER; footprint 2-PIN_SCREW-TERM_P200MIL -> connect-thru:1x2-SCREW-TERM_P200mil
- K1: footprint SHARP_SIP_SSR -> sharp:SHARP-SxxxSxx-SSR; moved to B.Cu
- LED1: value TXLED -> RED; footprint 0603(1608m)_led -> led:3mm-THRU-LED
- LED2: value RXLED -> GRN; footprint 0603(1608m)_led -> led:3mm-THRU-LED
- LED3: value ON -> 7-SEGMENT; footprint LED-5mm -> led:7-SEGMENT-4-DIGIT-DP+CLK_DIP16_W0.4in; moved to F.Cu
- LED4: value OFF -> 7-SEGMENT; footprint LED-5mm -> led:7-SEGMENT-4-DIGIT-DP+CLK_DIP16_W0.4in; moved to F.Cu
- LED5: value HOT -> RED; footprint LED-5mm -> led:3mm-THRU-LED; moved to F.Cu
- LED6: value 7-SEG_4-NUM-DISPLAY -> TXLED; footprint SF_4-DIGIT_7-SEGMENT_CC -> led:0603(1608m)-SM-LED; moved to F.Cu
- P1: footprint 2x3-array -> connect-thru:2x3-ARRAY_P100mil
- Q1, Q2, Q3, Q4, Q5: value MMBT4401 -> 2N7002; footprint SOT23 -> sot:SOT23
- R1: value opt10kΩ -> 10kΩ; footprint 0603(1608m) -> resistor:0603(1608m)-CHIP-RESISTOR
- R10, R11, R12, R14, R9: value opt10kΩ -> 330Ω; footprint 0603(1608m) -> resistor:0603(1608m)-CHIP-RESISTOR
- R13, R26, R27: value 180Ω -> 330Ω; footprint 0603(1608m) -> resistor:0603(1608m)-CHIP-RESISTOR
- R15, R16: value 180Ω -> 10kΩ; footprint 0603(1608m) -> resistor:0603(1608m)-CHIP-RESISTOR
- R17, R22, R23, R6: footprint 0603(1608m) -> resistor:0603(1608m)-CHIP-RESISTOR
- R18, R5: value 330Ω -> 10kΩ; footprint 0603(1608m) -> resistor:0603(1608m)-CHIP-RESISTOR
- R19: value 1kΩ -> 100Ω; footprint 0603(1608m) -> resistor:0603(1608m)-CHIP-RESISTOR
- R2, R3: value 4.7kΩ -> 10kΩ; footprint 0603(1608m) -> resistor:0603(1608m)-CHIP-RESISTOR
- R20: value 2.2kΩ -> 330Ω; footprint 0603(1608m) -> resistor:0603(1608m)-CHIP-RESISTOR
- R21: value 180Ω -> 10Ω; footprint 0603(1608m) -> resistor:1206(3216m)-CHIP-RESISTOR
- R24: value 180Ω -> 27Ω; footprint 0603(1608m) -> resistor:0603(1608m)-CHIP-RESISTOR
- R25: value 1kΩ -> 27Ω; footprint 0603(1608m) -> resistor:0603(1608m)-CHIP-RESISTOR
- R4: value 1MΩ -> 10kΩ; footprint 0603(1608m) -> resistor:0603(1608m)-CHIP-RESISTOR
- R7, R8: value 27Ω -> 330Ω; footprint 0603(1608m) -> resistor:0603(1608m)-CHIP-RESISTOR
- ROT1: value SET TEMP -> KNOB; footprint SF_ROTARY-ENCODER -> sparkfun:SF-ROTARY-ENCODER; moved to F.Cu
- S1: value START -> RST; footprint SPST_4-pin-thru -> switch:SPST-4-PIN_6mm_sm; moved to F.Cu
- TC1: footprint THERMOCOUPLE_MINI_PCC-SMP -> connect-thru:OMEGA-PCC-SMP_thermocouple-jack
- moved LED5 116.1 mm to (240.2, 121.2), turned to 0 degrees
- moved TC1 113.4 mm to (74.3, 41.9)
- moved R18 106.7 mm to (226.2, 149.0), turned to 0 degrees
- moved ROT1 100.8 mm to (94.0, 36.2), turned to 270 degrees
- moved LED3 100.3 mm to (123.8, 36.2)
- moved R16 96.9 mm to (218.8, 155.4), turned to 0 degrees
- moved R20 96.4 mm to (226.2, 145.9), turned to 0 degrees
- moved R19 86.5 mm to (235.4, 137.2)
- moved LED4 85.5 mm to (123.8, 51.4)
- moved R13 82.6 mm to (137.8, 45.7)
- moved R2 80.0 mm to (244.2, 132.2)
- moved R14 79.5 mm to (137.8, 43.8), turned to 0 degrees
- moved R17 78.6 mm to (238.8, 113.7)
- moved C1 78.0 mm to (253.5, 118.7), turned to 0 degrees
- moved C8 77.8 mm to (227.9, 136.8), turned to 0 degrees
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Connections:
- C10 pad 2: VCC -> Net-(C10-Pad2)
- C11 pad 1: N-0000067 -> GND
- C11 pad 2: GND -> Net-(C11-Pad2)
- C12 pad 2: N-0000052 -> Net-(C12-Pad2)
- C13 pad 2: N-0000039 -> VCC
- C2 pad 1: N-0000061 -> VCC
- C3 pad 1: GND -> +12V
- C3 pad 2: VCC -> GND
- C4 pad 1: N-0000064 -> GND
- C4 pad 2: N-0000061 -> Net-(C4-Pad2)
- C5 pad 2: N-0000064 -> Net-(C5-Pad2)
- C6 pad 1: GND -> Net-(C6-Pad1)
- C6 pad 2: VCC -> GND
- C9 pad 1: GND -> Net-(C9-Pad1)
- C9 pad 2: N-0000047 -> Net-(C9-Pad2)
- F1 pad 1: N-0000067 -> Net-(F1-Pad1)
- F1 pad 2: VCC -> Net-(C5-Pad2)
- IC1 pad 1: N-0000064 -> Net-(IC1-Pad1)
- IC1 pad 2: GND -> Net-(IC1-Pad2)
- IC1 pad 3: GND -> Net-(IC1-Pad3)
- IC1 pad 4: (no net) -> Net-(IC1-Pad4)
- IC1 pad 5: /TEMP -> Net-(IC1-Pad5)
- IC1 pad 6: /TEMP -> Net-(IC1-Pad6)
- IC1 pad 7: VCC -> Net-(IC1-Pad7)
- IC1 pad 8: N-0000061 -> GND
- IC2 pad 1: /STOP -> /DIG3
- IC2 pad 10: /LED_STOP -> /DIGA
- IC2 pad 11: /HEAT -> /DIGD
- IC2 pad 12: /SEGA -> /DIGC
- IC2 pad 13: /SEGG -> /DIGB
- IC2 pad 14: /SEGC -> /DIG1
- IC2 pad 15: /MOSI -> /DIG2
- IC2 pad 16: /MISO -> VCC
- IC2 pad 2: /SET -> /L0
- IC2 pad 3: GND -> /DIG0
- IC2 pad 4: VCC -> /L1
- IC2 pad 5: GND -> /DIG7
- IC2 pad 6: VCC -> /DIG4
- IC2 pad 7: /SEGF -> /DIG5
- IC2 pad 8: /SEGB -> GND
- IC2 pad 9: /LED_START -> /DIG6
- IC3 pad 1: /USART_RX -> GND
- IC3 pad 2: /RESET -> VCC
- IC3 pad 3: N-0000047 -> Net-(C4-Pad2)
- J1 pad 1: N-0000067 -> GND
- J1 pad 2: N-0000052 -> /AC1
- J2 pad 1: N-0000051 -> /HT
- J2 pad 2: N-0000049 -> GND
- K1 pad 1: N-0000051 -> /AC1
- K1 pad 2: N-0000049 -> /HT
- K1 pad 3: N-0000014 -> Net-(K1-Pad3)
- K1 pad 4: N-0000045 -> Net-(K1-Pad4)
- LED1 pad 1: N-0000043 -> /STAT_1
- LED1 pad 2: VCC -> Net-(LED1-Pad2)
- LED2 pad 1: N-0000037 -> Net-(LED1-Pad2)
- LED2 pad 2: VCC -> /STAT_1
- LED3 pad 1: N-000002 -> Net-(LED3-Pad1)
- LED3 pad 2: /LED_START -> Net-(LED3-Pad2)
- LED4 pad 1: N-000003 -> Net-(LED4-Pad1)
- LED4 pad 2: /LED_STOP -> Net-(LED4-Pad2)
- LED5 pad 1: N-0000050 -> Net-(LED5-Pad1)
- LED6 pad 1: N-000008 -> Net-(LED6-Pad1)
- LED6 pad 2: N-000007 -> VCC
- Q1 pad 1: N-0000012 -> /DIG7
- Q1 pad 3: N-0000019 -> Net-(LED3-Pad8)
- Q2 pad 1: N-0000053 -> /DIG6
- Q2 pad 3: N-0000045 -> Net-(LED3-Pad6)
- Q3 pad 1: N-0000030 -> /L1
- Q3 pad 3: N-0000020 -> Net-(LED3-Pad4)
- Q4 pad 1: N-0000016 -> /DIG5
- Q4 pad 3: N-0000055 -> Net-(LED3-Pad2)
- Q5 pad 1: N-0000018 -> /DIG4
- Q5 pad 3: N-0000056 -> Net-(LED3-Pad1)
- R1 pad 2: /RESET -> /DISP_CS
- R10 pad 1: /ENC_A -> /SEGE
- R10 pad 2: VCC -> Net-(IC1-Pad4)
- R11 pad 1: /ENC_B -> /SEGD
- R11 pad 2: VCC -> Net-(IC1-Pad3)
- R12 pad 1: /START -> /SEGC
- R12 pad 2: VCC -> Net-(IC1-Pad2)
- R13 pad 1: GND -> /SEGB
- R13 pad 2: N-000002 -> Net-(IC1-Pad1)
- R14 pad 1: /STOP -> /SEGA
- R14 pad 2: VCC -> Net-(IC1-Pad15)
- R15 pad 1: GND -> /ENC_A
- R15 pad 2: N-000003 -> VCC
- R16 pad 1: VCC -> /ENC_B
- R16 pad 2: N-0000014 -> VCC
- R17 pad 1: N-0000012 -> /ENC_C
- R17 pad 2: GND -> VCC
- R18 pad 1: N-0000050 -> /ENC_D
- R18 pad 2: N-0000045 -> VCC
- R19 pad 1: N-0000012 -> VCC
- R19 pad 2: /DIG1 -> Net-(K1-Pad3)
- R2 pad 1: N-0000044 -> GND
- R2 pad 2: N-0000061 -> Net-(IC1-Pad13)
- R20 pad 1: N-0000053 -> Net-(LED5-Pad1)
- R20 pad 2: /HEAT -> Net-(K1-Pad4)
- R21 pad 1: /SEGA -> Net-(C5-Pad2)
- R21 pad 2: N-000001 -> Net-(C6-Pad1)
- R22 pad 1: N-0000030 -> VCC
- R22 pad 2: GND -> /TEMP_CS
- R23 pad 1: N-0000053 -> VCC
- R23 pad 2: GND -> /RESET
- R24 pad 1: /SEGB -> Net-(C17-Pad2)
- R24 pad 2: N-000005 -> Net-(IC6-Pad9)
- R25 pad 1: N-0000030 -> Net-(C18-Pad2)
- R25 pad 2: /DIG2 -> Net-(IC6-Pad8)
- R26 pad 1: /SEGC -> Net-(IC6-Pad14)
- R26 pad 2: N-000006 -> Net-(LED6-Pad1)
- R27 pad 1: /MISO -> Net-(IC6-Pad7)
- R27 pad 2: N-000007 -> Net-(LED7-Pad1)
- R3 pad 1: N-0000062 -> /SW_TEMP
- R3 pad 2: N-0000064 -> VCC
- R4 pad 1: GND -> /SW_TIME
- R4 pad 2: N-0000062 -> VCC
- R5 pad 1: N-0000032 -> VCC
- R5 pad 2: N-0000043 -> Net-(IC1-Pad10)
- R6 pad 1: N-0000033 -> Net-(LED1-Pad2)
- R6 pad 2: N-0000037 -> /STAT_2
- R7 pad 1: N-0000052 -> /SEGDP
- R7 pad 2: N-0000046 -> Net-(IC1-Pad7)
- R8 pad 1: N-0000039 -> /SEGG
- R8 pad 2: N-0000038 -> Net-(IC1-Pad6)
- R9 pad 1: /SET -> /SEGF
- R9 pad 2: VCC -> Net-(IC1-Pad5)
- ROT1 pad 1: /SET -> /SW_TEMP
- S1 pad 2: /START -> /RESET
- TC1 pad 1: N-0000044 -> Net-(FB1-Pad1)
- TC1 pad 2: N-0000062 -> Net-(FB2-Pad1)
Routing:
- net GND: track 403.1 -> 0.00 mm, vias 34 -> 0
- net VCC: track 272.0 -> 0.00 mm, vias 5 -> 0
- net /STOP: track 117.7 -> 0.00 mm, vias 1 -> 0
- net /START: track 90.0 -> 0.00 mm, vias 1 -> 0
- net /RESET: track 76.7 -> 0.00 mm, vias 2 -> 0
- net /SET: track 57.9 -> 0.00 mm, vias 1 -> 0
- net /LED_STOP: track 52.3 -> 0.00 mm, vias 1 -> 0
- net /LED_START: track 49.4 -> 0.00 mm, vias 1 -> 0
- net /ENC_A: track 48.6 -> 0.00 mm, vias 1 -> 0
- net /ENC_B: track 43.5 -> 0.00 mm, vias 1 -> 0
- net /MOSI: track 37.9 -> 0.00 mm, vias 1 -> 0
- net /SCK: track 36.1 -> 0.00 mm, vias 1 -> 0
- net /USART_RX: track 35.3 -> 0.00 mm, vias 2 -> 0
- net /MISO: track 34.8 -> 0.00 mm, vias 1 -> 0
- net /USART_TX: track 28.9 -> 0.00 mm, vias 2 -> 0
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- removed copper zone on B.Cu, net GND
- removed copper zone on F.Cu, net GND
- removed copper zone on B.Cu, net N-0000049
- removed copper zone on F.Cu, net N-0000049
- removed copper zone on B.Cu, net N-0000051
- removed copper zone on F.Cu, net N-0000051
Other:
- board outline removed
- net class AC added: clearance 0.889, trace_width 2.032, via_dia 0.762, via_drill 0.381
- board text removed: "(so, um, don't like, touch it)"
- board text removed: "<-AC!!!"
- board text removed: "AC!!!"
- board text removed: "CUT OUT"
- board text removed: "github.com/mcous/reflow"
- board text removed: "github.com/mcous/reflow open source hardware cc by-sa 3.0 mjc 11/5/13"
- board text removed: "push to select"

Commit message: work on dimensions
Parts:
- moved TC1 36.4 mm to (99.1, 68.6), turned to 180 degrees
Changed lines of the file:
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@@
     (area 0 0 0 0)
     (thickness 1.6)
-    (drawings 5)
+    (drawings 7)
     (tracks 0)
     (zones 0)
@@
   )
   (module connect-thru:OMEGA-PCC-SMP_thermocouple-jack (layer F.Cu)
-    (at 74.295 41.91 90)
-    (fp_text reference TC1 (at 0 10.16 90) (layer F.SilkS)
-      (effects (font (size 0.762 0.762) (thickness 0.1524)))
-    )
-    (fp_text value THERMOCOUPLE (at 0 0 90) (layer F.SilkS) hide
+    (at 99.06 68.58 180)
+    (fp_text reference TC1 (at 0 10.16 180) (layer F.SilkS)
+      (effects (font (size 0.762 0.762) (thickness 0.1524)))
+    )
+    (fp_text value THERMOCOUPLE (at 0 0 180) (layer F.SilkS) hide
       (effects (font (size 0.762 0.762) (thickness 0.1524)))
     )
@@
     (fp_line (start -4.50088 8.001) (end 11.50112 8.001) (layer F.SilkS) (width 0.381))
     (fp_line (start 11.50112 -8.001) (end 11.50112 8.001) (layer F.SilkS) (width 0.381))
-    (pad 1 thru_hole circle (at -6.74878 -6.85038 90) (size 2.70002 2.70002) (drill 1.77038) (layers *.Cu *.Mask F.SilkS)
+    (pad 1 thru_hole circle (at -6.74878 -6.85038 180) (size 2.70002 2.70002) (drill 1.77038) (layers *.Cu *.Mask F.SilkS)
       (net 38 "Net-(FB1-Pad1)"))
-    (pad 2 thru_hole circle (at -6.74878 6.85038 90) (size 2.70002 2.70002) (drill 1.77038) (layers *.Cu *.Mask F.SilkS)
+    (pad 2 thru_hole circle (at -6.74878 6.85038 180) (size 2.70002 2.70002) (drill 1.77038) (layers *.Cu *.Mask F.SilkS)
       (net 39 "Net-(FB2-Pad1)"))
-    (pad "" thru_hole circle (at 6.74878 -7.85114 90) (size 2.70002 2.70002) (drill 1.77038) (layers *.Cu *.Mask F.SilkS))
-    (pad "" thru_hole circle (at 6.74878 7.85114 90) (size 2.70002 2.70002) (drill 1.77038) (layers *.Cu *.Mask F.SilkS))
+    (pad "" thru_hole circle (at 6.74878 -7.85114 180) (size 2.70002 2.70002) (drill 1.77038) (layers *.Cu *.Mask F.SilkS))
+    (pad "" thru_hole circle (at 6.74878 7.85114 180) (size 2.70002 2.70002) (drill 1.77038) (layers *.Cu *.Mask F.SilkS))
   )
   (module crystal:ABRACON-ABM2_xtal (layer F.Cu)
@@
       (net 36 /AC1))
   )
+  (dimension 88.9 (width 0.3) (layer Eco2.User)
+    (gr_text "3.5000 in" (at 128.905 22.78) (layer Eco2.User)
+      (effects (font (size 1.5 1.5) (thickness 0.3)))
+    )
+    (feature1 (pts (xy 173.355 28.575) (xy 173.355 21.43)))
+    (feature2 (pts (xy 84.455 28.575) (xy 84.455 21.43)))
+    (crossbar (pts (xy 84.455 24.13) (xy 173.355 24.13)))
+    (arrow1a (pts (xy 173.355 24.13) (xy 172.228496 24.716421)))
+    (arrow1b (pts (xy 173.355 24.13) (xy 172.228496 23.543579)))
+    (arrow2a (pts (xy 84.455 24.13) (xy 85.581504 24.716421)))
+    (arrow2b (pts (xy 84.455 24.13) (xy 85.581504 23.543579)))
+  )
+  (dimension 50.165 (width 0.3) (layer Eco2.User)
+    (gr_text "1.9750 in" (at 81.835 53.6575 270) (layer Eco2.User)
+      (effects (font (size 1.5 1.5) (thickness 0.3)))
+    )
+    (feature1 (pts (xy 85.09 78.74) (xy 80.485 78.74)))
+    (feature2 (pts (xy 85.09 28.575) (xy 80.485 28.575)))
+    (crossbar (pts (xy 83.185 28.575) (xy 83.185 78.74)))
+    (arrow1a (pts (xy 83.185 78.74) (xy 82.598579 77.613496)))
+    (arrow1b (pts (xy 83.185 78.74) (xy 83.771421 77.613496)))
+    (arrow2a (pts (xy 83.185 28.575) (xy 82.598579 29.701504)))
+    (arrow2b (pts (xy 83.185 28.575) (xy 83.771421 29.701504)))
+  )
   (dimension 38.1 (width 0.3) (layer Eco2.User)
